File: board/Simulation.kicad_sch (KiCad schematic)
At the start: 9 parts, among them U10 ${SIM.PARAMS}

Commit message: [23-5-2024] add micro sd card connector and MAX31856 Thermocouple driver
Parts:
- removed C3: 1n, Capacitor_SMD:C_01005_0402Metric_Pad0.57x0.30mm_HandSolder, symbol Device:C
- removed C6: 20n, Capacitor_SMD:C_01005_0402Metric_Pad0.57x0.30mm_HandSolder, symbol Device:C
- removed R10: 5.76k, Resistor_SMD:R_0805_2012Metric_Pad1.20x1.40mm_HandSolder, symbol Device:R_US
- removed R11: 2.21k, Resistor_SMD:R_0805_2012Metric_Pad1.20x1.40mm_HandSolder, symbol Device:R_US
- removed R12, R13: 1k, Resistor_SMD:R_0805_2012Metric_Pad1.20x1.40mm_HandSolder, symbol Device:R_US
- removed U10: ${SIM.PARAMS}, symbol Simulation_SPICE:OPAMP
- removed V1: VSIN, symbol Simulation_SPICE:VSIN
- removed V2: 5, symbol Simulation_SPICE:VDC
